Commit message: fix camera

File: urdf/tk8.urdf (robot description, URDF)
Before this commit: robot tk8, 9 links, 8 joints
Links:
- link base_servo_link: mass 0.049853330030012 -> 0.04985
- link bl_link: mass 0.0537442846179065 -> 0.05374
- link br_link: mass 0.0537442846179064 -> 0.05374
- link end_servo_link: mass 0.0688297822617074 -> 0.06883
- link fl_link: mass 0.0537442846179064 -> 0.05374
- link fr_link: mass 0.0537442846179065 -> 0.05374
Joints:
- joint base_servo_joint: origin xyz=-0.031274 -0.092587 0.11109 rpy=0 0 0 -> xyz=-0.03127 -0.09258 0.11109 rpy=0 0 0
- joint bl_joint: origin xyz=-0.078697 -0.195 0.031791 rpy=1.5708 0 1.5708 -> xyz=-0.0787 -0.195 0.03179 rpy=1.5708 0 1.5708
- joint br_joint: origin xyz=0.083303 -0.195 0.031791 rpy=1.5708 0 1.5708 -> xyz=0.0833 -0.195 0.03179 rpy=1.5708 0 1.5708
- joint camera_joint: origin xyz=0.0245 -0.1798 -0.051983 rpy=1.5708 0 0 -> xyz=0.0245 -0.1798 -0.05198 rpy=1.5708 0 0
- joint end_servo_joint: origin xyz=-0.00015257 0.03865 0.12837 rpy=-1.5708 0 0.00071232 -> xyz=-0.00015 0.03865 0.12837 rpy=-1.5708 0 0.00071
- joint fl_joint: origin xyz=-0.078697 -0.032 0.031791 rpy=1.5708 0 -1.5708 -> xyz=-0.0787 -0.032 0.03179 rpy=1.5708 0 -1.5708
- joint fr_joint: origin xyz=0.083303 -0.032 0.031791 rpy=1.5708 0 -1.5708 -> xyz=0.0833 -0.032 0.03179 rpy=1.5708 0 -1.5708
- joint lidar_joint: origin xyz=0.0023927 -0.01 0.045791 rpy=0 0 0 -> xyz=0.00239 -0.01 0.04579 rpy=0 0 0
